File: HARDWARE/uSupply/uSupply/Battery_Charging.kicad_sch (KiCad schematic)
At the start: 0 parts

Commit message: Added gitignore
same as before
Changed lines of the file:
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@@
   (symbol (lib_id "power:GND") (at 146.05 76.2 0) (unit 1)
     (in_bom yes) (on_board yes)
-    (property "Reference" "#PWR?" (id 0) (at 146.05 82.55 0)
+    (property "Reference" "#PWR02" (id 0) (at 146.05 82.55 0)
       (effects (font (size 1.27 1.27)) hide)
     )
-    (property "Value" "" (id 1) (at 146.177 80.5942 0))
+    (property "Value" "GND" (id 1) (at 146.177 80.5942 0))
     (property "Footprint" "" (id 2) (at 146.05 76.2 0)
       (effects (font (size 1.27 1.27)) hide)
