File: HARDWARE/uSupply/uSupply/SwitchingPowerPath.kicad_sch (KiCad schematic)
At the start: 19 parts

Commit message: Added gitignore
same as before
Parts:
- C1, C2, C3, C4, C5, C6, C7, C8, C9: renamed from C?; value (none) -> C
- D1: renamed from D?; value (none) -> D_Schottky
- L1: renamed from L?; value (none) -> L_Coupled
- R2, R3, R4, R5: renamed from R?; value (none) -> R
- U3: renamed from U?; value (none) -> U_MCP4131
- U4: renamed from U?; value (none) -> U_CS5171
- U5: renamed from U?; value (none) -> U_TC7600
