File: HARDWARE/mvSupply/AnalogPowerPath.kicad_sch (KiCad schematic)
At the start: 17 parts, among them U6 U_LM7805CT, U7 U_LT3080, U8 U_LM334

Commit message: Testing submodule retrieval
Committing to see if it will grab latest library commit
Parts:
- R10, R11, R12, R13, R14, R15, R16, R6, R7, R8, R9: footprint (none) -> master-vampire:R_AXIAL_L7mm_D2.6mm_P10mm_Horizontal
Changed lines of the file:
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@@
       (effects (font (size 1.27 1.27)) hide)
     )
-    (property "Footprint" "" (id 2) (at 187.198 100.33 0))
+    (property "Footprint" "master-vampire:R_AXIAL_L7mm_D2.6mm_P10mm_Horizontal" (id 2) (at 187.198 100.33 0)
+      (effects (font (size 1.27 1.27)) hide)
+    )
     (property "Datasheet" "" (id 3) (at 185.42 100.33 90))
     (property "Resistance" "10k" (id 4) (at 186.7662 101.4984 90)
@@
       (effects (font (size 1.27 1.27)) hide)
     )
-    (property "Footprint" "" (id 2) (at 102.87 74.422 0))
+    (property "Footprint" "master-vampire:R_AXIAL_L7mm_D2.6mm_P10mm_Horizontal" (id 2) (at 102.87 74.422 0)
+      (effects (font (size 1.27 1.27)) hide)
+    )
     (property "Datasheet" "" (id 3) (at 102.87 76.2 90))
     (property "Resistance" "10k" (id 4) (at 110.49 74.93 0)
@@
       (effects (font (size 1.27 1.27)) hide)
     )
-    (property "Footprint" "" (id 2) (at 102.87 71.882 0))
+    (property "Footprint" "master-vampire:R_AXIAL_L7mm_D2.6mm_P10mm_Horizontal" (id 2) (at 102.87 71.882 0)
+      (effects (font (size 1.27 1.27)) hide)
+    )
     (property "Datasheet" "" (id 3) (at 102.87 73.66 90))
     (property "Resistance" "10k" (id 4) (at 110.49 72.39 0)
@@
       (effects (font (size 1.27 1.27)) hide)
     )
-    (property "Footprint" "" (id 2) (at 102.87 69.342 0))
+    (property "Footprint" "master-vampire:R_AXIAL_L7mm_D2.6mm_P10mm_Horizontal" (id 2) (at 102.87 69.342 0)
+      (effects (font (size 1.27 1.27)) hide)
+    )
     (property "Datasheet" "" (id 3) (at 102.87 71.12 90))
     (property "Resistance" "10k" (id 4) (at 110.49 69.85 0)
@@
       (effects (font (size 1.27 1.27)) hide)
     )
-    (property "Footprint" "" (id 2) (at 102.87 66.802 0))
+    (property "Footprint" "master-vampire:R_AXIAL_L7mm_D2.6mm_P10mm_Horizontal" (id 2) (at 102.87 66.802 0)
+      (effects (font (size 1.27 1.27)) hide)
+    )
     (property "Datasheet" "" (id 3) (at 102.87 68.58 90))
     (property "Resistance" "10k" (id 4) (at 110.49 67.31 0)
@@
       (effects (font (size 1.27 1.27)) hide)
     )
-    (property "Footprint" "" (id 2) (at 102.87 64.262 0))
+    (property "Footprint" "master-vampire:R_AXIAL_L7mm_D2.6mm_P10mm_Horizontal" (id 2) (at 102.87 64.262 0)
+      (effects (font (size 1.27 1.27)) hide)
+    )
     (property "Datasheet" "" (id 3) (at 102.87 66.04 90))
     (property "Resistance" "10k" (id 4) (at 110.49 64.77 0)
@@
       (effects (font (size 1.27 1.27)) hide)
     )
-    (property "Footprint" "" (id 2) (at 102.87 61.722 0))
+    (property "Footprint" "master-vampire:R_AXIAL_L7mm_D2.6mm_P10mm_Horizontal" (id 2) (at 102.87 61.722 0)
+      (effects (font (size 1.27 1.27)) hide)
+    )
     (property "Datasheet" "" (id 3) (at 102.87 63.5 90))
     (property "Resistance" "10k" (id 4) (at 110.49 62.23 0)
@@
       (effects (font (size 1.27 1.27)) hide)
     )
-    (property "Footprint" "" (id 2) (at 102.87 59.182 0))
+    (property "Footprint" "master-vampire:R_AXIAL_L7mm_D2.6mm_P10mm_Horizontal" (id 2) (at 102.87 59.182 0)
+      (effects (font (size 1.27 1.27)) hide)
+    )
     (property "Datasheet" "" (id 3) (at 102.87 60.96 90))
     (property "Resistance" "10k" (id 4) (at 110.49 59.69 0)
@@
       (effects (font (size 1.27 1.27)) hide)
     )
-    (property "Footprint" "" (id 2) (at 102.87 56.642 0))
+    (property "Footprint" "master-vampire:R_AXIAL_L7mm_D2.6mm_P10mm_Horizontal" (id 2) (at 102.87 56.642 0)
+      (effects (font (size 1.27 1.27)) hide)
+    )
     (property "Datasheet" "" (id 3) (at 102.87 58.42 90))
     (property "Resistance" "10k" (id 4) (at 110.49 57.15 0)
@@
       (effects (font (size 1.27 1.27)) hide)
     )
-    (property "Footprint" "" (id 2) (at 102.87 54.102 0))
+    (property "Footprint" "master-vampire:R_AXIAL_L7mm_D2.6mm_P10mm_Horizontal" (id 2) (at 102.87 54.102 0)
+      (effects (font (size 1.27 1.27)) hide)
+    )
     (property "Datasheet" "" (id 3) (at 102.87 55.88 90))
     (property "Resistance" "10k" (id 4) (at 110.49 54.61 0)
@@
       (effects (font (size 1.27 1.27)) hide)
     )
-    (property "Footprint" "" (id 2) (at 102.87 51.562 0))
+    (property "Footprint" "master-vampire:R_AXIAL_L7mm_D2.6mm_P10mm_Horizontal" (id 2) (at 102.87 51.562 0)
+      (effects (font (size 1.27 1.27)) hide)
+    )
     (property "Datasheet" "" (id 3) (at 102.87 53.34 90))
     (property "Resistance" "10k" (id 4) (at 110.49 52.07 0)
