File: HARDWARE/mvSupply/Interface.kicad_sch (KiCad schematic)
At the start: 35 parts, among them SW3 SW_2-Pin_SHIELD, SW4 SW_2-Pin_SHIELD, SW5 SW_2-Pin_SHIELD, SW6 SW_2-Pin_SHIELD

Commit message: Testing submodule retrieval
Committing to see if it will grab latest library commit
Parts:
- R17, R18, R19, R20, R21, R22, R23, R24, R25, R26, R27, R28, R29, R30, R31, R32, R33, R34: footprint (none) -> master-vampire:R_AXIAL_L7mm_D2.6mm_P10mm_Horizontal
Changed lines of the file:
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@@
       (effects (font (size 1.27 1.27)) hide)
     )
-    (property "Footprint" "" (id 2) (at 197.358 26.67 0))
+    (property "Footprint" "master-vampire:R_AXIAL_L7mm_D2.6mm_P10mm_Horizontal" (id 2) (at 197.358 26.67 0)
+      (effects (font (size 1.27 1.27)) hide)
+    )
     (property "Datasheet" "" (id 3) (at 195.58 26.67 90))
     (property "Resistance" "10k" (id 4) (at 196.9262 27.8384 90)
@@
       (effects (font (size 1.27 1.27)) hide)
     )
-    (property "Footprint" "" (id 2) (at 204.978 26.67 0))
+    (property "Footprint" "master-vampire:R_AXIAL_L7mm_D2.6mm_P10mm_Horizontal" (id 2) (at 204.978 26.67 0)
+      (effects (font (size 1.27 1.27)) hide)
+    )
     (property "Datasheet" "" (id 3) (at 203.2 26.67 90))
     (property "Resistance" "10k" (id 4) (at 204.5462 27.8384 90)
@@
       (effects (font (size 1.27 1.27)) hide)
     )
-    (property "Footprint" "" (id 2) (at 101.6 86.36 0))
+    (property "Footprint" "" (id 2) (at 101.6 86.36 0)
+      (effects (font (size 1.27 1.27)) hide)
+    )
     (property "Datasheet" "" (id 3) (at 101.6 86.36 0))
     (property "Manufacturer" "Harvatek Corporation" (id 4) (at 101.6 72.39 0)
@@
       (effects (font (size 1.27 1.27)) hide)
     )
-    (property "Footprint" "" (id 2) (at 33.528 30.48 0))
+    (property "Footprint" "master-vampire:R_AXIAL_L7mm_D2.6mm_P10mm_Horizontal" (id 2) (at 33.528 30.48 0)
+      (effects (font (size 1.27 1.27)) hide)
+    )
     (property "Datasheet" "" (id 3) (at 31.75 30.48 90))
     (property "Resistance" "10k" (id 4) (at 33.0962 31.6484 90)
@@
       (effects (font (size 1.27 1.27)) hide)
     )
-    (property "Footprint" "" (id 2) (at 66.548 30.48 0))
+    (property "Footprint" "master-vampire:R_AXIAL_L7mm_D2.6mm_P10mm_Horizontal" (id 2) (at 66.548 30.48 0)
+      (effects (font (size 1.27 1.27)) hide)
+    )
     (property "Datasheet" "" (id 3) (at 64.77 30.48 90))
     (property "Resistance" "10k" (id 4) (at 66.1162 31.6484 90)
@@
       (effects (font (size 1.27 1.27)) hide)
     )
-    (property "Footprint" "" (id 2) (at 25.4 41.402 0))
+    (property "Footprint" "master-vampire:R_AXIAL_L7mm_D2.6mm_P10mm_Horizontal" (id 2) (at 25.4 41.402 0)
+      (effects (font (size 1.27 1.27)) hide)
+    )
     (property "Datasheet" "" (id 3) (at 25.4 43.18 90))
     (property "Resistance" "10k" (id 4) (at 22.86 40.64 0)
@@
       (effects (font (size 1.27 1.27)) hide)
     )
-    (property "Footprint" "" (id 2) (at 71.12 41.402 0))
+    (property "Footprint" "master-vampire:R_AXIAL_L7mm_D2.6mm_P10mm_Horizontal" (id 2) (at 71.12 41.402 0)
+      (effects (font (size 1.27 1.27)) hide)
+    )
     (property "Datasheet" "" (id 3) (at 71.12 43.18 90))
     (property "Resistance" "10k" (id 4) (at 68.58 40.64 0)
@@
       (effects (font (size 1.27 1.27)) hide)
     )
-    (property "Footprint" "" (id 2) (at 33.528 71.12 0))
+    (property "Footprint" "master-vampire:R_AXIAL_L7mm_D2.6mm_P10mm_Horizontal" (id 2) (at 33.528 71.12 0)
+      (effects (font (size 1.27 1.27)) hide)
+    )
     (property "Datasheet" "" (id 3) (at 31.75 71.12 90))
     (property "Resistance" "10k" (id 4) (at 33.0962 72.2884 90)
@@
       (effects (font (size 1.27 1.27)) hide)
     )
-    (property "Footprint" "" (id 2) (at 66.548 71.12 0))
+    (property "Footprint" "master-vampire:R_AXIAL_L7mm_D2.6mm_P10mm_Horizontal" (id 2) (at 66.548 71.12 0)
+      (effects (font (size 1.27 1.27)) hide)
+    )
     (property "Datasheet" "" (id 3) (at 64.77 71.12 90))
     (property "Resistance" "10k" (id 4) (at 66.1162 72.2884 90)
@@
       (effects (font (size 1.27 1.27)) hide)
     )
-    (property "Footprint" "" (id 2) (at 25.4 82.042 0))
+    (property "Footprint" "master-vampire:R_AXIAL_L7mm_D2.6mm_P10mm_Horizontal" (id 2) (at 25.4 82.042 0)
+      (effects (font (size 1.27 1.27)) hide)
+    )
     (property "Datasheet" "" (id 3) (at 25.4 83.82 90))
     (property "Resistance" "10k" (id 4) (at 22.86 81.28 0)
@@
       (effects (font (size 1.27 1.27)) hide)
     )
-    (property "Footprint" "" (id 2) (at 71.12 82.042 0))
+    (property "Footprint" "master-vampire:R_AXIAL_L7mm_D2.6mm_P10mm_Horizontal" (id 2) (at 71.12 82.042 0)
+      (effects (font (size 1.27 1.27)) hide)
+    )
     (property "Datasheet" "" (id 3) (at 71.12 83.82 90))
     (property "Resistance" "10k" (id 4) (at 68.58 81.28 0)
@@
       (effects (font (size 1.27 1.27)) hide)
     )
-    (property "Footprint" "" (id 2) (at 103.378 72.39 0))
+    (property "Footprint" "master-vampire:R_AXIAL_L7mm_D2.6mm_P10mm_Horizontal" (id 2) (at 103.378 72.39 0)
+      (effects (font (size 1.27 1.27)) hide)
+    )
     (property "Datasheet" "" (id 3) (at 101.6 72.39 90))
     (property "Resistance" "330" (id 4) (at 96.52 73.66 90)
@@
       (effects (font (size 1.27 1.27)) hide)
     )
-    (property "Footprint" "" (id 2) (at 116.078 72.39 0))
+    (property "Footprint" "master-vampire:R_AXIAL_L7mm_D2.6mm_P10mm_Horizontal" (id 2) (at 116.078 72.39 0)
+      (effects (font (size 1.27 1.27)) hide)
+    )
     (property "Datasheet" "" (id 3) (at 114.3 72.39 90))
     (property "Resistance" "330" (id 4) (at 109.22 73.66 90)
@@
       (effects (font (size 1.27 1.27)) hide)
     )
-    (property "Footprint" "" (id 2) (at 128.778 72.39 0))
+    (property "Footprint" "master-vampire:R_AXIAL_L7mm_D2.6mm_P10mm_Horizontal" (id 2) (at 128.778 72.39 0)
+      (effects (font (size 1.27 1.27)) hide)
+    )
     (property "Datasheet" "" (id 3) (at 127 72.39 90))
     (property "Resistance" "330" (id 4) (at 121.92 73.66 90)
@@
       (effects (font (size 1.27 1.27)) hide)
     )
-    (property "Footprint" "" (id 2) (at 141.478 72.39 0))
+    (property "Footprint" "master-vampire:R_AXIAL_L7mm_D2.6mm_P10mm_Horizontal" (id 2) (at 141.478 72.39 0)
+      (effects (font (size 1.27 1.27)) hide)
+    )
     (property "Datasheet" "" (id 3) (at 139.7 72.39 90))
     (property "Resistance" "330" (id 4) (at 134.62 73.66 90)
@@
       (effects (font (size 1.27 1.27)) hide)
     )
-    (property "Footprint" "" (id 2) (at 39.878 124.46 0))
+    (property "Footprint" "master-vampire:R_AXIAL_L7mm_D2.6mm_P10mm_Horizontal" (id 2) (at 39.878 124.46 0)
+      (effects (font (size 1.27 1.27)) hide)
+    )
     (property "Datasheet" "" (id 3) (at 38.1 124.46 90))
     (property "Resistance" "10k" (id 4) (at 39.4462 125.6284 90)
@@
       (effects (font (size 1.27 1.27)) hide)
     )
-    (property "Footprint" "" (id 2) (at 52.578 124.46 0))
+    (property "Footprint" "master-vampire:R_AXIAL_L7mm_D2.6mm_P10mm_Horizontal" (id 2) (at 52.578 124.46 0)
+      (effects (font (size 1.27 1.27)) hide)
+    )
     (property "Datasheet" "" (id 3) (at 50.8 124.46 90))
     (property "Resistance" "10k" (id 4) (at 52.1462 125.6284 90)
@@
       (effects (font (size 1.27 1.27)) hide)
     )
-    (property "Footprint" "" (id 2) (at 65.278 124.46 0))
+    (property "Footprint" "master-vampire:R_AXIAL_L7mm_D2.6mm_P10mm_Horizontal" (id 2) (at 65.278 124.46 0)
+      (effects (font (size 1.27 1.27)) hide)
+    )
     (property "Datasheet" "" (id 3) (at 63.5 124.46 90))
     (property "Resistance" "10k" (id 4) (at 64.8462 125.6284 90)
@@
       (effects (font (size 1.27 1.27)) hide)
     )
-    (property "Footprint" "" (id 2) (at 77.978 124.46 0))
+    (property "Footprint" "master-vampire:R_AXIAL_L7mm_D2.6mm_P10mm_Horizontal" (id 2) (at 77.978 124.46 0)
+      (effects (font (size 1.27 1.27)) hide)
+    )
     (property "Datasheet" "" (id 3) (at 76.2 124.46 90))
     (property "Resistance" "10k" (id 4) (at 77.5462 125.6284 90)
@@
       (effects (font (size 1.27 1.27)) hide)
     )
-    (property "Footprint" "" (id 2) (at 114.3 86.36 0))
+    (property "Footprint" "" (id 2) (at 114.3 86.36 0)
+      (effects (font (size 1.27 1.27)) hide)
+    )
     (property "Datasheet" "" (id 3) (at 114.3 86.36 0))
     (property "Manufacturer" "Harvatek Corporation" (id 4) (at 114.3 72.39 0)
@@
       (effects (font (size 1.27 1.27)) hide)
     )
-    (property "Footprint" "" (id 2) (at 127 86.36 0))
+    (property "Footprint" "" (id 2) (at 127 86.36 0)
+      (effects (font (size 1.27 1.27)) hide)
+    )
     (property "Datasheet" "" (id 3) (at 127 86.36 0))
     (property "Manufacturer" "Harvatek Corporation" (id 4) (at 127 72.39 0)
@@
       (effects (font (size 1.27 1.27)) hide)
     )
-    (property "Footprint" "" (id 2) (at 139.7 86.36 0))
+    (property "Footprint" "" (id 2) (at 139.7 86.36 0)
+      (effects (font (size 1.27 1.27)) hide)
+    )
     (property "Datasheet" "" (id 3) (at 139.7 86.36 0))
     (property "Manufacturer" "Harvatek Corporation" (id 4) (at 139.7 72.39 0)
