File: HARDWARE/mvSupply/SwitchingPowerPath.kicad_sch (KiCad schematic)
At the start: 18 parts, among them U3 U_MCP4131, U4 U_CS5171, U5 U_TC7600

Commit message: Testing submodule retrieval
Committing to see if it will grab latest library commit
Parts:
- R3, R4, R5: footprint (none) -> master-vampire:R_AXIAL_L7mm_D2.6mm_P10mm_Horizontal
Changed lines of the file:
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@@
       (effects (font (size 1.27 1.27)) hide)
     )
-    (property "Footprint" "" (id 2) (at 93.98 156.972 0))
+    (property "Footprint" "master-vampire:R_AXIAL_L7mm_D2.6mm_P10mm_Horizontal" (id 2) (at 93.98 156.972 0)
+      (effects (font (size 1.27 1.27)) hide)
+    )
     (property "Datasheet" "" (id 3) (at 93.98 158.75 90))
     (property "Resistance" "10k" (id 4) (at 93.98 156.083 0)
@@
       (effects (font (size 1.27 1.27)) hide)
     )
-    (property "Footprint" "" (id 2) (at 102.108 143.51 0))
+    (property "Footprint" "master-vampire:R_AXIAL_L7mm_D2.6mm_P10mm_Horizontal" (id 2) (at 102.108 143.51 0)
+      (effects (font (size 1.27 1.27)) hide)
+    )
     (property "Datasheet" "" (id 3) (at 100.33 143.51 90))
     (property "Resistance" "10k" (id 4) (at 101.6762 144.6784 90)
@@
       (effects (font (size 1.27 1.27)) hide)
     )
-    (property "Footprint" "" (id 2) (at 77.978 30.48 0))
+    (property "Footprint" "master-vampire:R_AXIAL_L7mm_D2.6mm_P10mm_Horizontal" (id 2) (at 77.978 30.48 0)
+      (effects (font (size 1.27 1.27)) hide)
+    )
     (property "Datasheet" "" (id 3) (at 76.2 30.48 90))
     (property "Resistance" "10k" (id 4) (at 77.5462 31.6484 90)
@@
       (effects (font (size 1.27 1.27)) hide)
     )
-    (property "Footprint" "" (id 2) (at 63.5 69.342 0))
+    (property "Footprint" "" (id 2) (at 63.5 69.342 0)
+      (effects (font (size 1.27 1.27)) hide)
+    )
     (property "Datasheet" "" (id 3) (at 63.5 71.12 90))
     (property "Resistance" "10k" (id 4) (at 63.5 68.453 0)
@@
       (effects (font (size 1.27 1.27)) hide)
     )
-    (property "Footprint" "" (id 2) (at 128.27 80.01 90))
+    (property "Footprint" "" (id 2) (at 128.27 80.01 90)
+      (effects (font (size 1.27 1.27)) hide)
+    )
     (property "Datasheet" "" (id 3) (at 128.27 80.01 90))
     (property "Inductance" "33uH" (id 4) (at 129.3622 81.1784 90)
@@
       (effects (font (size 1.27 1.27)) hide)
     )
-    (property "Footprint" "" (id 2) (at 146.05 80.01 90))
+    (property "Footprint" "" (id 2) (at 146.05 80.01 90)
+      (effects (font (size 1.27 1.27)) hide)
+    )
     (property "Datasheet" "" (id 3) (at 146.05 80.01 90))
     (property "Inductance" "33uH" (id 4) (at 147.1422 81.1784 90)
